File: 05_ElettroScheme/reversePendulum-System/mv-scheme.sch (EAGLE design)
At the start: 15 parts, among them IC1 7805T, IC2 L298, X1 GLX-S-88M, X2 GLX-S-88M

Commit message: control presentation and elettronic draw
Parts:
- removed X1: GLX-S-88M, con-kycon:GLX-S-88M
- added MOT-CON: GLX-S-88M, con-kycon:GLX-S-88M
- renumbered X2 to MPU-CON
Connections:
- net +5V: now also MOT-CON.3; no longer X1.3
- net ENA: now also MOT-CON.4; no longer X1.4
- net ENB: now also MOT-CON.5; no longer X1.5
- net GND: now also MOT-CON.6; no longer X1.6
- net MOT+: now also MOT-CON.1, MOT-CON.2; no longer X1.1, X1.2
- net MOT-: now also MOT-CON.7, MOT-CON.8; no longer X1.7, X1.8
Other:
- moved on the sheet: CON_A-B, CON_C-D, CON_D-C, CON_E-F, CON_F-E, IC2, PWR, R1, START/STOP, TARATURA
